File: hvawg.kicad_sch (KiCad schematic)
At the start: 90 parts, among them J1 Conn_01x04_Pin, J10 Conn_01x01_Pin, J2 Conn_01x04_Pin, J3 Conn_01x04_Pin, J4 Conn_01x04_Pin, J5 Conn_01x04_Pin, J6 Conn_01x04_Pin, J7 Conn_01x04_Pin, J8 Conn_01x04_Pin, J9 Conn_01x08_Pin, Q1 IRF730, Q3 IRF9610, U1 L7805, U2 74HC595D,110, U3 DAC0808LCMX/NOPB, U4 NE5532, U6 LM8261, U7 LM8261, U8 NE5532

Commit message: Fix Q3 source/drain swap in design files; regenerate gerbers
Connections:
- net levelshift_out: now also Q3.2 (D); no longer Q3.3 (S)
- net at RV1.2, U6.4 (-): now also Q3.3 (S); no longer Q3.2 (D)

Commit message: new board
Parts:
- removed J10: Conn_01x01_Pin, Connector_PinSocket_2.54mm:PinSocket_1x01_P2.54mm_Horizontal, symbol Connector:Conn_01x01_Pin
- added C32: DNP, Capacitor_SMD:C_1206_3216Metric, symbol Device:C
- added D4, D5: BZT52C12, Diode_SMD:D_SOD-123, symbol Device:D_Zener
- added HS1: Wakefield 272-AB, Library:Heatsink_Wakefield_272-AB, symbol Mechanical:Heatsink_Pad_2Pin
- added R26: 3.3k, Resistor_SMD:R_0402_1005Metric, symbol Device:R
- added R27: 820, Resistor_SMD:R_0402_1005Metric, symbol Device:R
- added R28: 100k, Resistor_SMD:R_0402_1005Metric, symbol Device:R
- added R29: 1M, Resistor_SMD:R_0402_1005Metric, symbol Device:R
- added R30: 22k, Resistor_SMD:R_2512_6332Metric, symbol Device:R
- added R31: 4.7k, Resistor_SMD:R_2512_6332Metric, symbol Device:R
- added R32: DNP, Resistor_SMD:R_1206_3216Metric, symbol Device:R
- added TP10, TP11, TP12, TP9: TestPoint, TestPoint:TestPoint_Pad_D1.5mm, symbol Connector:TestPoint
- added TP6, TP7, TP8: TestPoint, TestPoint:TestPoint_Keystone_5005-5009_Compact, symbol Connector:TestPoint
- added unit 2 of U4
- added unit 2 of U8
- C24: MPN (none) -> CL31B106KAHNNNE; Note (none) -> Samsung CL31B106KAHNNNE 10 uF 10% 25 V X7R (-55 to +125 C) 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
- J7: value Conn_01x04_Pin -> Conn_01x07_Pin; footprint Library:PinSocket_1x04_P2.54mm_Horizontal_flipped -> Library:PinSocket_1x07_P2.54mm_Horizontal_flipped; symbol Connector:Conn_01x04_Pin -> Connector:Conn_01x07_Pin
- J8: value Conn_01x04_Pin -> Conn_01x07_Pin; footprint Connector_PinSocket_2.54mm:PinSocket_1x04_P2.54mm_Horizontal -> Connector_PinSocket_2.54mm:PinSocket_1x07_P2.54mm_Horizontal; symbol Connector:Conn_01x04_Pin -> Connector:Conn_01x07_Pin
- J9: footprint Connector_PinHeader_2.54mm:PinHeader_1x08_P2.54mm_Vertical -> Library:PhoenixContact_MC_1,5_8-G-3.5_1x08_P3.50mm_Horizontal_EdgeNotch; MPN (none) -> 1844278; Note (none) -> Phoenix Contact MC 1,5/8-G-3,5 (1844278) 8-pin 3.50 mm PCB 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
- Q1, Q3: footprint Package_TO_SOT_THT:TO-220-3_Vertical -> Library:TO-220-3_Vertical_HV
- R21: footprint Resistor_THT:R_Axial_Power_L25.0mm_W9.0mm_P10.16mm_Vertical -> Library:TO-220-2_Horizontal_LTO50; MPN (none) -> LTO050F10001JTE3; Note (none) -> Vishay LTO 50 (LTO050F10001JTE3, the BOM part; the flat foo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
- RV1: value 3k -> 1k
Connections:
- net +100V: now also J5.1 (Pin_1), J6.1 (Pin_1), J9.5 (Pin_5); no longer J5.2 (Pin_2), J6.2 (Pin_2), J9.6 (Pin_6)
- net +12V: now also J9.2 (Pin_2); no longer J9.3 (Pin_3)
- net -100+12V: now also J5.4 (Pin_4), J6.4 (Pin_4), J9.8 (Pin_8), TP11.1; no longer J5.3 (Pin_3), J6.3 (Pin_3), J9.7 (Pin_7)
- net -100V: now also J5.3 (Pin_3), J6.3 (Pin_3), J9.7 (Pin_7), TP12.1; no longer J5.4 (Pin_4), J6.4 (Pin_4), J9.8 (Pin_8)
- net -12V: now also J9.3 (Pin_3); no longer J9.4 (Pin_4)
- net GND: now also J5.2 (Pin_2), J6.2 (Pin_2), J7.2 (Pin_2), J7.4 (Pin_4), J7.6 (Pin_6), J8.2 (Pin_2), J8.4 (Pin_4), J8.6 (Pin_6), J9.4 (Pin_4), J9.6 (Pin_6), C32.2, HS1.1, HS1.2, R27.2, U4.5 (+), U8.5 (+); no longer J5.1 (Pin_1), J6.1 (Pin_1), J9.2 (Pin_2), J9.5 (Pin_5), RV2.2
- net output_post: now reaches JP10.1 (A), JP11.1 (A), JP8.1 (A), JP9.1 (A)
- net output_post: now also R31.2, TP6.1; no longer Q1.2 (D), R21.1, TP5.1
- net at J7.3 (Pin_3), J8.3 (Pin_3): now also JP9.2 (B); no longer JP10.2 (B)
- net at C14.1, C15.1, R12.2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: now also R30.1; no longer U8.3 (+)
- net at RV2.3: now also RV2.2, R27.1
- net at JP6.1 (A): now also R26.1; no longer RV1.1
- net at Q1.1 (G), R18.1, U7.1: now also D4.1 (K), R28.1, TP9.1
- net at Q1.3 (S), R22.1, R23.2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: now also D4.2 (A), R28.2, TP10.1
- net at Q3.1 (G), U6.1: now also D5.2 (A), R29.2, TP7.1
- net at Q3.3 (S), RV1.2, U6.4 (-): now also RV1.3, D5.1 (K), R29.1, TP8.1
- new net: J7.5 (Pin_5), J8.5 (Pin_5), JP10.2 (B)
- new net: U4.6 (-), U4.7
- new net: J7.7 (Pin_7), J8.7 (Pin_7), JP11.2 (B)
- new net: Q1.2 (D), R21.1, R31.1, R32.1, TP5.1
- new net: C32.1, R32.2
- new net: R26.2, RV1.1
- new net: R30.2, U8.3 (+)
- new net: U8.6 (-), U8.7
Other:
- note added: "C32 if fitted: >=250 V rated"
- note added: "J7/J8 output bus: 1,3,5,7 = OUT1..OUT4 2,4,6 = GND/shield"
- note removed: "for cable ground shield"

Commit message: all of the V2 changes: schematic changes, labels, regenerated gerbers, etc
Parts:
- C24: Note Samsung CL31B106KAHNNNE 10 uF 10% 25 V X7R (-55 to +125 C) 1206, LCSC C14860 (JLC extended part): must be X7R 125 C because C24 sits about 7 mm from the HS1 heat sink; do not fit the May-BOM X5R 85 C CL31A106KBHNNNE (C13585). Floating 12 V rail (-100V to -100+12V), so 25 V is 2x margin. -> Samsung CL31B106KAHNNNE 10 uF 10% 25 V X7R (-55 to +125 C) 1206, LCSC C14860 (JLC extended part): must be X7R 125 C because C24 sits about 7 mm from the HS1 heat sink; do not fit the X5R 85 C CL31A106KBHNNNE (C13585) from the original (V1) JLC BOM. Floating 12 V rail (-100V to -100+12V), so 25 V is 2x margin.
- C26, C27: symbol Device:C -> Device:C_Polarized
- C32, R32: now in the parts list
- D4, D5: MPN (none) -> BZT52C12
- Q1: symbol Device:Q_NMOS_GDS -> Transistor_FET:Q_NMOS_GDS
- Q3: symbol Device:Q_PMOS_GDS -> Transistor_FET:Q_PMOS_GDS
- R1, R10, R11, R17, R2, R3, R4, R5, R6, R7, R8, R9: value 2.7k -> 2.74k; MPN (none) -> RT0402BRE072K74L
- R26: MPN (none) -> 0402WGF3301TCE
- R27: MPN (none) -> 0402WGF8200TCE
- R28: MPN (none) -> 0402WGF1003TCE
- R29: MPN (none) -> 0402WGF1004TCE
- R31: MPN (none) -> CRGP2512F4K7; Note (none) -> TE CRGP2512F4K7 4.7k 1% 2W (70C) 500V pulse-rated thick fil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
- U1: value L7805 -> L78M05ABDT-TR; MPN (none) -> L78M05ABDT-TR
- U2: value 74HC595D,110 -> 74HCT595D,118; symbol 74xx:74HC595 -> 74xx:74HCT595; MPN (none) -> 74HCT595D,118
- U3: Note (none) -> DAC0808 output compliance is only guaranteed from -5V to +0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
Connections:
- net +5V: now reaches C2.1, C3.1, C4.1, C5.1, C6.1, JP1.2 (B), R4.1, R7.1, TP1.1, U1.3 (OUT), U2.10 (~{SRCLR}), U2.16 (VCC), U3.1 (VCC)
Other:
- note added: "V2: 110k 0.5W 200V 2010 part, 0.20W at 150V, 0.13W at 120V"
- note added: "V2: R19/R23 not fitted, so the mirror is R17/R22 = 2.74k/75 = 36.5x."
- note added: "V2: R26 3.3k + RV1 1k (rheostat) = 3.3-4.3k. RV1 centers the output: about 3.65k at R_bottom 1.11k, preset 4.3k. Mirror R17/R22 = 2.74k/75 = 36.5x."
- note added: "V2: RV2 1k rheostat + R27 820 = R_bottom 0.82-1.82k. RV2 sets the gain (110k+R_bottom)/R_bottom. Preset 1.11k for gain 100."
